Commit message: Add ros2_control integration and Gazebo simulation support

File: src/arduinobot_description/urdf/arduinobot.urdf.xacro (robot description, xacro)
@@ -1,230 +1,182 @@
 <?xml version="1.0"?>
-<robot name="arduinobot" xmlns:xacro="http://www.ros.org/wiki/xacro">
-  <xacro:arg />
-  <xacro:property name="PI" value="3.14159"/>
-  <xacro:property name="effort" value="30.0"/>
-  <xacro:property name="velocity" value="10.0"/>
-  <xacro:macro name="default_inertia" params="mass">
-    <inertial>
-      <origin xyz="0 0 0" rpy="0 0 0"/>
-      <mass value="${mass}"/>
-      <inertia ixx="1.0" ixy="0.0" ixz="0.0"
-              iyy="1.0" iyz="0.0"
-              izz="1.0"/>
-    </inertial>
-  </xacro:macro>
-  <link name="world"/>
-  <link name="base_link">
-      <xacro:default_inertia mass="1.0"/>
-      <visual>
-          <origin rpy="0 0 0" xyz="-0.5 -0.5 0"/>
-          <geometry>
-              <mesh filename="package://arduinobot_description/meshes/basement.STL" scale="0.01 0.01 0.01"/>
-          </geometry>
-      </visual>
-      <collision>
-          <origin rpy="0 0 0" xyz="-0.5 -0.5 0"/>
-          <geometry>
-              <mesh filename="package://arduinobot_description/meshes/basement.STL" scale="0.01 0.01 0.01"/>
-          </geometry>
-      </collision>
-  </link>
-  <joint name="virtual_joint" type="fixed">
-    <parent link="world"/>
-    <child link="base_link"/>
-    <origin rpy="0 0 0" xyz="0 0 0"/>
-  </joint>
-  <link name="base_plate">
-    <xacro:default_inertia mass="0.1"/>
-    <visual>
-      <origin rpy="0 0 0" xyz="-0.39 -0.39 -0.56"/>
-      <geometry>
-        <mesh filename="package://arduinobot_description/meshes/base_plate.STL"
-              scale="0.01 0.01 0.01"/>
-      </geometry>
-    </visual>
-    <collision>
-      <origin rpy="0 0 0" xyz="-0.39 -0.39 -0.56"/>
-      <geometry>
-        <mesh filename="package://arduinobot_description/meshes/base_plate.STL"
-              scale="0.01 0.01 0.01"/>
-      </geometry>
-    </collision>
-  </link>
-  <joint name="joint_1" type="revolute">
-    <parent link="base_link"/>
-    <child link="base_plate"/>
-    <axis xyz="0 0 1"/>
-    <origin rpy="0 0 0" xyz="0 0 0.307"/>
-    <limit lower="-${PI/2}" upper="${PI/2}"
-          effort="${effort}" velocity="${velocity}"/>
-  </joint>
-  <link name="forward_drive_arm">
-      <xacro:default_inertia mass="0.1"/>
-      <visual>
-          <origin rpy=" 0 -${PI / 2} ${PI / 2}" xyz="0.19 0.06 -0.08"/>
-          <geometry>
-              <mesh filename="package://arduinobot_description/meshes/forward_drive_arm.STL" scale="0.01 0.01 0.01"/>
-          </geometry>
-      </visual>
-      <collision>
-          <origin rpy=" 0 -${PI / 2} ${PI / 2}" xyz="0.19 0.06 -0.08"/>
-          <geometry>
-              <mesh filename="package://arduinobot_description/meshes/forward_drive_arm.STL" scale="0.01 0.01 0.01"/>
-          </geometry>
-      </collision>
-  </link>
-  <joint name="joint_2" type="revolute">
-    <parent link="base_plate"/>
-    <child link="forward_drive_arm"/>
-    <axis xyz="1 0 0"/>
-    <origin rpy="0 0 0" xyz="-0.02 0 0.35"/>
-    <limit lower="-${PI/2}" upper="${PI/2}"
-          effort="${effort}" velocity="${velocity}"/>
-  </joint>
-  <link name="horizontal_arm">
-    <xacro:default_inertia mass="0.1"/>
-    <visual>
-      <origin rpy="${PI/2} 0 ${PI/2}" xyz="-0.03 -0.4 -0.06"/>
-      <geometry>
-        <mesh filename="package://arduinobot_description/meshes/horizontal_arm.STL" scale="0.01 0.01 0.01"/>
-      </geometry>
-    </visual>
-    <collision>
-      <origin rpy="${PI/2} 0 ${PI/2}" xyz="-0.03 -0.4 -0.06"/>
-      <geometry>
-        <mesh filename="package://arduinobot_description/meshes/horizontal_arm.STL" scale="0.01 0.01 0.01"/>
-      </geometry>
-    </collision>
-  </link>
-  <joint name="joint_3" type="revolute">
-    <parent link="forward_drive_arm"/>
-    <child link="horizontal_arm"/>
-    <axis xyz="1 0 0"/>
-    <origin rpy="0 0 0" xyz="0 0 0.8"/>
-    <limit lower="-${PI/2}" upper="${PI/2}"
-          effort="${effort}" velocity="${velocity}"/>
-  </joint>
-  <link name="claw_support">
-    <xacro:default_inertia mass="0.05"/>
-    <visual>
-      <origin rpy="0 0 ${PI/2}" xyz="0 0.03 0.15"/>
-      <geometry>
-        <mesh filename="package://arduinobot_description/meshes/claw_support.STL" scale="0.01 0.01 0.01"/>
-      </geometry>
-    </visual>
-    <collision>
-      <origin rpy="0 0 ${PI/2}" xyz="0 0.03 0.15"/>
-      <geometry>
-        <mesh filename="package://arduinobot_description/meshes/claw_support.STL" scale="0.01 0.01 0.01"/>
-      </geometry>
-    </collision>
-  </link>
-  <joint name="horizontal_arm_to_claw_support" type="fixed">
-    <parent link="horizontal_arm"/>
-    <child link="claw_support"/>
-    <origin rpy="0 0 0" xyz="0 0.82 0"/>
-  </joint>
-  <link name="gripper_right">
-    <xacro:default_inertia mass="0.01"/>
-    <visual>
-    <origin xyz="-0.1 0.5 0.1" rpy="0 0 -${PI/2}"/>
-      <geometry>
-        <mesh filename="package://arduinobot_description/meshes/right_finger.STL" scale="0.01 0.01 0.01"/>
-      </geometry>
-    </visual>
-    <collision>
-      <origin xyz="-0.1 0.5 0.1" rpy="0 0 -${PI/2}"/>
-      <geometry>
-        <mesh filename="package://arduinobot_description/meshes/right_finger.STL" scale="0.01 0.01 0.01"/>
-      </geometry>
-    </collision>
-  </link>
-  <link name="gripper_left">
-    <xacro:default_inertia mass="0.01"/>
-    <visual>
-    <origin xyz="-0.04 0.5 -0.01" rpy="0 0 -${PI/2}"/>
-      <geometry>
-        <mesh filename="package://arduinobot_description/meshes/left_finger.STL" scale="0.01 0.01 0.01"/>
-      </geometry>
-    </visual>
-    <collision>
-      <origin xyz="-0.04 0.5 -0.01" rpy="0 0 -${PI/2}"/>
-      <geometry>
-        <mesh filename="package://arduinobot_description/meshes/left_finger.STL" scale="0.01 0.01 0.01"/>
-      </geometry>
-    </collision>
-  </link>
-  <joint name="joint_4" type="revolute">
-    <parent link="claw_support"/>
-    <child link="gripper_right"/>
-    <axis xyz="0 0 1"/>
-    <origin rpy="0 0 0" xyz="-0.04 0.13 -0.1"/>
-    <limit lower="-${PI/2}" upper="0.0"
-          effort="${effort}" velocity="${velocity}"/>
-  </joint>
-  <joint name="joint_5" type="revolute">
-    <parent link="claw_support"/>
-    <child link="gripper_left"/>
-    <axis xyz="0 0 1"/>
-    <origin rpy="0 0 0" xyz="-0.22 0.13 -0.1"/>
-    <mimic joint="joint_4" multiplier="-1"/>
-    <limit lower="0.0" upper="${PI/2}"
-          effort="${effort}" velocity="${velocity}"/>
-  </joint>
-  <link name="rgb_camera">
-      <xacro:default_inertia mass="0.001"/>
-      <visual>
-          <origin rpy="-1.57 0 -1.57" xyz="-0.1 0.125 0.15"/>
-          <geometry>
-              <mesh filename="package://arduinobot_description/meshes/pi_camera.STL" scale="0.01 0.01 0.01"/>
-          </geometry>
-      </visual>
-      <collision>
-          <origin rpy="-1.57 0 -1.57" xyz="-0.1 0.125 0.15"/>
-          <geometry>
-              <mesh filename="package://arduinobot_description/meshes/pi_camera.STL" scale="0.01 0.01 0.01"/>
-          </geometry>
-      </collision>
-  </link>
-  <joint name ="rgb_camera_joint" type="fixed">
-      <parent link="base_link"/>
-      <child link = "rgb_camera"/>
-      <origin xyz="0 0.45 0.2" rpy="0 -0.5 1.57"/>
-  </joint>
-  <gazebo reference="rgb_camera">
-    <sensor name="camera" type="camera">
-      <gz_frame_id>rgb_camera</gz_frame_id>
-      <always_on>true</always_on>
-      <update_rate>30</update_rate>
-      <visualize>true</visualize>
-      <topic>image_raw</topic>
-      <camera name="camera">
-        <horizontal_fov>1.15</horizontal_fov>
-        <image>
-          <width>2304</width>
-          <height>1296</height>
-          <format>R8G8B8</format>
-        </image>
-        <distortion>
-          <k1>0.0</k1>
-          <k2>0.0</k2>
-          <k3>0.0</k3>
-          <p1>0.0</p1>
-          <p2>0.0</p2>
-          <center>0.5 0.5</center>
-        </distortion>
-        <clip>
-          <near>0.01</near>
-          <far>100</far>
-        </clip>
-      </camera>
-    </sensor>
-  </gazebo>
-  <gazebo reference="rgb_camera">
-    <plugin
-        filename="gz-sim-sensors-system"
-        name="gz::sim::systems::Sensors">
-    </plugin>
-  </gazebo>
+<robot xmlns:xacro="http://www.ros.org/wiki/xacro" name="arduinobot">
+    <!-- Start GZ or Ignition depending on ROS 2 Version -->
+    <xacro:arg name="is_ignition" default="true"/>
+    <!-- Include Gazebo Parameters -->
+    <xacro:include filename="$(find arduinobot_description)/urdf/arduinobot_gazebo.xacro" />
+    <!-- Include ros2_control Plugins -->
+    <xacro:include filename="$(find arduinobot_description)/urdf/arduinobot_ros2_control.xacro" />
+    <!-- Useful XACRO Variables (Properties) -->
+    <xacro:property name="PI" value="3.14159265359" />
+    <xacro:property name="effort" value="30.0" />
+    <xacro:property name="velocity" value="10.0" />
+    <!-- Useful Macros -->
+    <xacro:macro name="default_inertial" params="mass">
+        <inertial>
+            <origin xyz="0 0 0" rpy="0 0 0"/>
+            <mass value="${mass}" />
+            <inertia ixx="1.0" ixy="0.0" ixz="0.0"
+                     iyy="1.0" iyz="0.0"
+                     izz="1.0" />
+        </inertial>
+    </xacro:macro>
+    <!-- Links -->
+    <link name="world"/>
+    <link name="base_link">
+        <xacro:default_inertial mass="1.0"/>
+        <visual>
+            <origin rpy="0 0 0" xyz="-0.5 -0.5 0"/>
+            <geometry>
+                <mesh filename="package://arduinobot_description/meshes/basement.STL" scale="0.01 0.01 0.01"/>
+            </geometry>
+        </visual>
+        <collision>
+            <origin rpy="0 0 0" xyz="-0.5 -0.5 0"/>
+            <geometry>
+                <mesh filename="package://arduinobot_description/meshes/basement.STL" scale="0.01 0.01 0.01"/>
+            </geometry>
+        </collision>
+    </link>
+    <link name="base_plate">
+        <xacro:default_inertial mass="0.1"/>
+        <visual>
+            <origin rpy="0 0 0" xyz="-0.39 -0.39 -0.56"/>
+            <geometry>
+                <mesh filename="package://arduinobot_description/meshes/base_plate.STL" scale="0.01 0.01 0.01"/>
+            </geometry>
+        </visual>
+        <collision>
+            <origin rpy="0 0 0" xyz="-0.39 -0.39 -0.56"/>
+            <geometry>
+                <mesh filename="package://arduinobot_description/meshes/base_plate.STL" scale="0.01 0.01 0.01"/>
+            </geometry>
+        </collision>
+    </link>
+    <link name="forward_drive_arm">
+        <xacro:default_inertial mass="0.1"/>
+        <visual>
+            <origin rpy=" 0 -${PI / 2} ${PI / 2}" xyz="0.19 0.06 -0.08"/>
+            <geometry>
+                <mesh filename="package://arduinobot_description/meshes/forward_drive_arm.STL" scale="0.01 0.01 0.01"/>
+            </geometry>
+        </visual>
+        <collision>
+            <origin rpy=" 0 -${PI / 2} ${PI / 2}" xyz="0.19 0.06 -0.08"/>
+            <geometry>
+                <mesh filename="package://arduinobot_description/meshes/forward_drive_arm.STL" scale="0.01 0.01 0.01"/>
+            </geometry>
+        </collision>
+    </link>
+    <link name="horizontal_arm">
+        <xacro:default_inertial mass="0.1"/>
+        <visual>
+            <origin rpy="${PI / 2} 0 ${PI / 2}" xyz="-0.03 -0.4 -0.06"/>
+            <geometry>
+                <mesh filename="package://arduinobot_description/meshes/horizontal_arm.STL" scale="0.01 0.01 0.01"/>
+            </geometry>
+        </visual>
+        <collision>
+            <origin rpy="${PI / 2} 0 ${PI / 2}" xyz="-0.03 -0.4 -0.06"/>
+            <geometry>
+                <mesh filename="package://arduinobot_description/meshes/horizontal_arm.STL" scale="0.01 0.01 0.01"/>
+            </geometry>
+        </collision>
+    </link>
+    <link name="claw_support">
+        <xacro:default_inertial mass="0.05"/>
+        <visual>
+            <origin rpy="0 0 ${PI / 2}" xyz="0 -0.05 -0.15"/>
+            <geometry>
+                <mesh filename="package://arduinobot_description/meshes/claw_support.STL" scale="0.01 0.01 0.01"/>
+            </geometry>
+        </visual>
+        <collision>
+            <origin rpy="0 0 ${PI / 2}" xyz="0 -0.05 -0.15"/>
+            <geometry>
+                <mesh filename="package://arduinobot_description/meshes/claw_support.STL" scale="0.01 0.01 0.01"/>
+            </geometry>
+        </collision>
+    </link>
+    <link name="gripper_right">
+        <xacro:default_inertial mass="0.01"/>
+        <visual>
+            <origin rpy="0 0 -${PI / 2}" xyz="-0.1 0.50 -0.1"/>
+            <geometry>
+                <mesh filename="package://arduinobot_description/meshes/right_finger.STL" scale="0.01 0.01 0.01"/>
+            </geometry>
+        </visual>
+        <collision>
+            <origin rpy="0 0 -${PI / 2}" xyz="-0.1 0.50 -0.1"/>
+            <geometry>
+                <mesh filename="package://arduinobot_description/meshes/right_finger.STL" scale="0.01 0.01 0.01"/>
+            </geometry>
+        </collision>
+    </link>
+    <link name="gripper_left">
+        <xacro:default_inertial mass="0.01"/>
+        <visual>
+            <origin rpy="0 0 -${PI / 2}" xyz="-0.04 0.50 -0.1"/>
+            <geometry>
+                <mesh filename="package://arduinobot_description/meshes/left_finger.STL" scale="0.01 0.01 0.01"/>
+            </geometry>
+        </visual>
+        <collision>
+            <origin rpy="0 0 -${PI / 2}" xyz="-0.04 0.50 -0.1"/>
+            <geometry>
+                <mesh filename="package://arduinobot_description/meshes/left_finger.STL" scale="0.01 0.01 0.01"/>
+            </geometry>
+        </collision>
+    </link>
+    <!-- Joints -->
+    <joint name="virtual_joint" type="fixed">
+        <parent link="world"/>
+        <child link="base_link"/>
+        <origin xyz="0 0 0" rpy="0 0 0"/>
+    </joint>
+    <joint name ="joint_1" type="revolute">
+        <parent link="base_link"/>
+        <child link = "base_plate"/>
+        <origin xyz="0 0 0.307"/>
+        <axis xyz="0 0 1"/>
+        <limit lower="-${PI / 2}" upper="${PI / 2}"
+               effort="${effort}" velocity="${velocity}"/>
+    </joint>
+    <joint name ="joint_2" type="revolute">
+        <parent link="base_plate"/>
+        <child link = "forward_drive_arm"/>
+        <origin xyz="-0.02 0 0.35"/>
+        <axis xyz="1 0 0"/>
+        <limit lower="-${PI / 2}" upper="${PI / 2}"
+                effort="${effort}" velocity="${velocity}"/>
+    </joint>
+    <joint name ="joint_3" type="revolute">
+        <parent link="forward_drive_arm"/>
+        <child link = "horizontal_arm"/>
+        <origin xyz="0 0 0.8"/>
+        <axis xyz="1 0 0"/>
+        <limit lower="-${PI / 2}" upper="${PI / 2}"
+               effort="${effort}" velocity="${velocity}"/>
+    </joint>
+    <joint name ="horizontal_arm_to_claw_support" type="fixed">
+        <parent link="horizontal_arm"/>
+        <child link = "claw_support"/>
+        <origin xyz="0 0.82 0"/>
+    </joint>
+    <joint name ="joint_4" type="revolute">
+        <parent link="claw_support"/>
+        <child link = "gripper_right"/>
+        <origin xyz="-0.04 0.13 -0.1"/>
+        <axis xyz="0 0 1"/>
+        <limit lower="-${PI / 2}" upper="0.0"
+               effort="${effort}" velocity="${velocity}"/>
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